File: NRF_HEX_V1.1/NRF_HEX_V1.1.kicad_sch (KiCad schematic)
At the start: 12 parts, among them Y1 32Mhz, Y2 32.768Mhz

Commit message: hex pcb updated and power management system added
Parts:
- removed Y1: 32Mhz, Crystal:Crystal_SMD_0603-2Pin_6.0x3.5mm, symbol Device:Crystal_Small
- added C19: 0.1uF, Capacitor_SMD:C_0402_1005Metric_Pad0.74x0.62mm_HandSolder, symbol Device:C_Small
- added C22, C23: 1uF, Capacitor_SMD:C_0402_1005Metric_Pad0.74x0.62mm_HandSolder, symbol Device:C_Small
- added C24: 22uF, Capacitor_SMD:C_0402_1005Metric_Pad0.74x0.62mm_HandSolder, symbol Device:C_Small
- added J1: Conn_01x03_Socket, Connector_PinHeader_2.54mm:PinHeader_1x03_P2.54mm_Vertical, symbol Connector:Conn_01x03_Socket
- added J2: Conn_01x06_Socket, Connector_PinSocket_2.54mm:PinSocket_1x06_P2.54mm_Vertical, symbol Connector:Conn_01x06_Socket
- added J3: Conn_01x04_Socket, Connector_PinSocket_2.54mm:PinSocket_1x04_P2.54mm_Vertical, symbol Connector:Conn_01x04_Socket
- added MK1: ICS-43434, Sensor_Audio:InvenSense_ICS-43434-6_3.5x2.65mm, symbol Sensor_Audio:ICS-43434
- added R7: 10k, Resistor_SMD:R_0402_1005Metric_Pad0.72x0.64mm_HandSolder, symbol Device:R_Small_US
- added R8: 100k, Resistor_SMD:R_0402_1005Metric_Pad0.72x0.64mm_HandSolder, symbol Device:R_Small_US
- added U4: ESP32-S3-WROOM-1, RF_Module:ESP32-S3-WROOM-1, symbol RF_Module:ESP32-S3-WROOM-1
- added U7: 74AHCT125, Package_DIP:DIP-14_W7.62mm_SMDSocket_SmallPads, symbol 74xx:74AHCT125
- C3: value 12pF -> 1uF
- C4: value 12pF -> 0.1uF
Connections:
- net GND: now also C4.1, U1.1 (GND), U1.2 (GND), U1.26 (GND), U1.43 (GND), C19.2, C22.2, C23.1, C24.1, J2.3 (Pin_3), J3.4 (Pin_4), MK1.2 (LR), MK1.3 (GND), R8.2, U4.1 (GND), U4.40 (GND), U4.41 (GND)
- net +3.3V: now reaches U1.3 (VDD)
- net +3.3V: now also C4.2, C19.1, C22.1, C24.2, J2.2 (Pin_2), J3.1 (Pin_1), MK1.5 (VDD), R7.2, U4.2 (3V3)
- net IO_3: now reaches U1.33 (P17)
- net IO_3: now also J1.3 (Pin_3)
- net IO_2: now reaches U1.34 (P18)
- net IO_2: now also J1.2 (Pin_2)
- net IO_1: now reaches U1.35 (P19)
- net IO_1: now also J1.1 (Pin_1)
- net IN_1: now reaches U1.37 (Reset/P21)
- net IN_1: now also J2.6 (Pin_6)
- net SCL: now reaches U1.38 (SCLK)
- net SCL: now also J2.5 (Pin_5)
- net SDA: now reaches U1.39 (SDIO)
- net SDA: now also J2.4 (Pin_4)
- new net: C23.2, R7.1, U4.3 (EN)
- new net +5V: U7.14 (VCC)
- new net D+: U4.14 (USB_D+)
- new net D-: U4.13 (USB_D-)
- new net MIC_SCK: MK1.4 (SCK), U4.21 (IO13)
- new net MIC_SD: MK1.6 (SD), R8.1, U4.22 (IO14)
- new net MIC_WS: MK1.1 (WS), U4.20 (IO12)
- new net RX: J3.2 (Pin_2), U4.36 (RXD0)
- new net TX: J3.3 (Pin_3), U4.37 (TXD0)
- new net VSYS: J2.1 (Pin_1)
Other:
- added sheet LED (LED.kicad_sch)
- note added: "ESP32_S3"
- note added: "I2C_BREAKOUT"
- note added: "Level_Converter"
- note added: "MB-N2_Module(NRF)"
- note added: "Microphone_Module"
- note added: "NRF_GPIO"
- note added: "UART"
- moved on the sheet: C1, C2, C4, C5, C6, C7, L1, L2, U1, Y2
